File: carzycar.kicad_sch (KiCad schematic)
At the start: 18 parts, among them IC1 RZ7889, IC2 RZ7889, J1 SWD header, J2 Conn_01x06_Pin, J3 Conn_01x06_Pin, SW1 Push_Button, U1 STM32C031C4Tx, U2 TMCS1100A3QDR, U3 TMCS1100A3QDR

Commit message: update only layout missing
Parts:
- added BZ1: Buzzer, Buzzer_Beeper:Buzzer_12x9.5RM7.6, symbol Device:Buzzer
- added C10: 1n, Capacitor_SMD:C_0805_2012Metric, symbol Device:C
- added C11, C13: 10u, Capacitor_SMD:C_0805_2012Metric, symbol Device:C
- added C12, C14, C15, C5, C7, C8, C9: 100n, Capacitor_SMD:C_0805_2012Metric, symbol Device:C
- added C6: 10n, Capacitor_SMD:C_0805_2012Metric, symbol Device:C
- added D1, D2: LED, LED_SMD:LED_0805_2012Metric, symbol Device:LED
- added J10: Conn_01x02_Socket, Connector_PinHeader_2.54mm:PinHeader_1x02_P2.54mm_Vertical, symbol Connector:Conn_01x02_Socket
- added J4, J5, J6, J7, J8: VL53L0X, Connector_PinHeader_2.54mm:PinHeader_1x05_P2.54mm_Vertical, symbol Connector:Conn_01x05_Pin
- added J9: Conn_01x02_Socket, Connector_AMASS:AMASS_XT30U-F_1x02_P5.0mm_Vertical, symbol Connector:Conn_01x02_Socket
- added Q1: 2N3904, Package_TO_SOT_THT:TO-92_Inline, symbol Transistor_BJT:2N3904
- added R10, R16, R17, R8: 10k, Resistor_SMD:R_0805_2012Metric, symbol Device:R
- added R11: 68R, Resistor_SMD:R_0805_2012Metric, symbol Device:R
- added R12: 47k, Resistor_SMD:R_0805_2012Metric, symbol Device:R
- added R13, R14: 330R, Resistor_SMD:R_0805_2012Metric, symbol Device:R
- added R15: 1k, Resistor_SMD:R_0805_2012Metric, symbol Device:R
- added R6, R7: 4k7, Resistor_SMD:R_0805_2012Metric, symbol Device:R
- added R9: 33k, Resistor_SMD:R_0805_2012Metric, symbol Device:R
- added U4: TCA9548APWR, Package_SO:TSSOP-24_4.4x7.8mm_P0.65mm, symbol Interface_Expansion:TCA9548APWR
- added U5: MPU-6500, MPU-6500:QFN40P300X300X95-25N, symbol MPU-6500:MPU-6500
- added U6: QRE1113GR, OptoDevice:OnSemi_CASE100CY, symbol Sensor_Proximity:QRE1113GR
- added U7: LD1117V33, Package_TO_SOT_THT:TO-220-3_Horizontal_TabDown, symbol Regulator_Linear:LD1117V33
- added V1: 1N4148, Diode_THT:D_DO-35_SOD27_P7.62mm_Horizontal, symbol diode_AilM:1N4148_P7
- C1, C2, C4: footprint (none) -> Capacitor_SMD:C_0805_2012Metric
- C3: footprint Package_LCC:PLCC-44_16.6x16.6mm_P1.27mm -> Capacitor_THT:CP_Radial_D8.0mm_P3.50mm
- J1: footprint Package_DFN_QFN:QFN-20-1EP_5x5mm_P0.65mm_EP3.35x3.35mm -> Connector_PinHeader_2.54mm:PinHeader_1x05_P2.54mm_Vertical
- J2, J3: footprint Package_DFN_QFN:QFN-20-1EP_5x5mm_P0.65mm_EP3.35x3.35mm -> Connector_PinHeader_2.54mm:PinHeader_1x06_P2.54mm_Vertical
- R1: footprint Button_Switch_THT:SW_PUSH_6mm -> Resistor_SMD:R_0805_2012Metric
- R2, R3, R4, R5: footprint SOIC8_D_TEX -> Resistor_SMD:R_0805_2012Metric
- U2, U3: footprint SOIC8_D_TEX -> TMCS1100A1:SOIC8_D_TEX
Connections:
- net +3.3V: now also BZ1.1 (+), C12.1, C13.1, C5.1, C6.1, C8.1, R11.1, R12.1, R13.1, R16.2, R6.1, R7.2, R8.1, U4.24 (VCC), U4.3 (~{RESET}), U5.13 (VDD), U5.8 (VDDIO), U7.2 (VO), V1.1 (C)
- net +7.4V: now also C11.1, J9.2 (Pin_2), R9.2, U7.3 (VI)
- net GND: now also C10.2, C11.2, C12.2, C13.2, C14.1, C15.2, C5.2, C6.2, C7.2, C8.2, C9.1, D1.1 (K), D2.1 (K), J10.2 (Pin_2), J4.1 (Pin_1), J5.1 (Pin_1), J6.1 (Pin_1), J7.1 (Pin_1), J8.1 (Pin_1), J9.1 (Pin_1), Q1.1 (E), R10.2, R17.2, U4.1 (A0), U4.12 (GND), U4.2 (A1), U4.21 (A2), U5.11 (FSYNC), U5.18 (GND), U5.20 (RESV_2), U6.2 (K), U6.4, U7.1 (GND)
- net NRST: now also C14.2
- net Vref: no longer U3.6 (VREF)
- net V_BAT: now reaches U1.13 (PA2)
- net V_BAT: now also C9.2, R10.1, R9.1
- net CS: now reaches U1.15 (PA4)
- net CS: now also R8.2, U5.22 (NCS)
- net SCK: now reaches U1.16 (PA5)
- net SCK: now also U5.23 (SCL/SCLK)
- net SDO: now reaches U1.17 (PA6)
- net SDO: now also U5.9 (AD0/SDO)
- net SDI: now reaches U1.18 (PA7)
- net SDI: now also U5.24 (SDA/SDI)
- net INT: now reaches U1.21 (PB2)
- net INT: now also U5.12 (INT)
- net at U1.34 (PA12): now also R14.1
- net at U1.42 (PB3): now also R15.1
- net at U1.45 (PB6): now also J10.1 (Pin_1)
- net SCL: now reaches U1.47 (PB8)
- net SCL: now also R7.1, U4.22 (SCL)
- net SDA: now reaches U1.48 (PB9)
- net SDA: now also R6.2, U4.23 (SDA)
- new net: J6.2 (Pin_2), U4.7 (SC1)
- new net: J6.3 (Pin_3), U4.6 (SD1)
- new net: D2.2 (A), R14.2
- new net: D1.2 (A), R13.2
- new net: BZ1.2 (-), Q1.3 (C), V1.2 (A)
- new net: Q1.2 (B), R15.2
- new net: J7.2 (Pin_2), U4.9 (SC2)
- new net: J7.3 (Pin_3), U4.8 (SD2)
- new net: J4.2 (Pin_2), U4.11 (SC3)
- new net: J4.3 (Pin_3), U4.10 (SD3)
- new net: J8.2 (Pin_2), U4.5 (SC0)
- new net: J8.3 (Pin_3), U4.4 (SD0)
- new net: R11.2, U6.1 (A)
- new net: C7.1, U5.10 (REGOUT)
- new net: J5.2 (Pin_2), U4.14 (SC4)
- new net: J5.3 (Pin_3), U4.13 (SD4)
- new net LAP: C10.1, R12.2, U6.3
- new net Vref1: C15.1, R16.1, R17.1, U3.6 (VREF)
Other:
- note added: "Battery Voltage"
- note added: "Distance Sensors"
- note added: "IMU"
- note added: "Lap Sensor BOTTOM SIDE"
- note added: "Voltage Regulator"

Commit message: Add files via upload
Parts:
- removed C10: 1n, Capacitor_SMD:C_0805_2012Metric, symbol Device:C
- removed R11: 68R, Resistor_SMD:R_0805_2012Metric, symbol Device:R
- removed R12: 47k, Resistor_SMD:R_0805_2012Metric, symbol Device:R
- removed U6: QRE1113GR, OptoDevice:OnSemi_CASE100CY, symbol Sensor_Proximity:QRE1113GR
- added HNP1, HNP10, HNP2, HNP3, HNP4, HNP5, HNP6, HNP7, HNP8, HNP9: NPH, MountingHole:MountingHole_2.2mm_M2, symbol basic_AilM:MountingHole
- added M1, M2: Motor_DC, minimouse:N20_with_encoder, symbol Motor:Motor_DC
- BZ1: DISTRIBUTOR (none) -> LCSC; MANUFACTURER (none) -> XHXDZ; ORDER_NO (none) -> C49246932; PART_NO (none) -> TMB12A12; PRICE_UNIT (none) -> 0.1884
- C1, C12, C14, C15, C2, C4, C5, C7, C8, C9: DISTRIBUTOR (none) -> LCSC; MANUFACTURER (none) -> YAGEO; ORDER_NO (none) -> C49678; PART_NO (none) -> CC0805KRX7R9BB104; PRICE_UNIT (none) -> 0.019
- C11, C13: DISTRIBUTOR (none) -> LCSC; MANUFACTURER (none) -> muRata; ORDER_NO (none) -> C440198; PART_NO (none) -> GRM21BR61H106KE43L; PRICE_UNIT (none) -> 0.182
- C3: DISTRIBUTOR (none) -> LCSC; MANUFACTURER (none) -> KNSCHA; ORDER_NO (none) -> C2831775; PART_NO (none) -> 03EC0575; PRICE_UNIT (none) -> 0.0415
- C6: DISTRIBUTOR (none) -> LCSC; MANUFACTURER (none) -> CCTC; ORDER_NO (none) -> C282728; PART_NO (none) -> TCC0805X7R103K500DT; PRICE_UNIT (none) -> 0.0061
- D1, D2: DISTRIBUTOR (none) -> LCSC; MANUFACTURER (none) -> XINGLIGHT; ORDER_NO (none) -> C965799; PART_NO (none) -> XL-1608SURC-06; PRICE_UNIT (none) -> 0.0034
- IC1, IC2: DISTRIBUTOR (none) -> LCSC; MANUFACTURER (none) -> MSKSEMI; ORDER_NO (none) -> C22462543; PART_NO (none) -> RZ7889-MS; PRICE_UNIT (none) -> 0.4336
- J1, J10, J2, J3, J4, J5, J6, J7, J8: DISTRIBUTOR (none) -> LCSC; MANUFACTURER (none) -> Ckmtw; ORDER_NO (none) -> C124377; PART_NO (none) -> B-2100S40P-A110; PRICE_UNIT (none) -> 0.2542
- J9: DISTRIBUTOR (none) -> LCSC; MANUFACTURER (none) -> AMASS; ORDER_NO (none) -> C99102; PART_NO (none) -> XT30U-F; PRICE_UNIT (none) -> 0.1920
- Q1: DISTRIBUTOR (none) -> LCSC; MANUFACTURER (none) -> onsemi; ORDER_NO (none) -> C124482; PART_NO (none) -> 2N3904BU; PRICE_UNIT (none) -> 0.0945
- R1, R10, R16, R17, R2, R3, R8: DISTRIBUTOR (none) -> LCSC; MANUFACTURER (none) -> UNI-ROYAL; ORDER_NO (none) -> C17414; PART_NO (none) -> 0805W8F1002T5E; PRICE_UNIT (none) -> 0.0032
- R13, R14: DISTRIBUTOR (none) -> LCSC; MANUFACTURER (none) -> UNI-ROYAL; ORDER_NO (none) -> C17630; PART_NO (none) -> 0805W8F3300T5E; PRICE_UNIT (none) -> 0.0042
- R15: DISTRIBUTOR (none) -> LCSC; MANUFACTURER (none) -> YAGEO; ORDER_NO (none) -> C95781; PART_NO (none) -> RC0805FR-071KL; PRICE_UNIT (none) -> 0.0029
- R4, R5: DISTRIBUTOR (none) -> LCSC; MANUFACTURER (none) -> FOJAN; ORDER_NO (none) -> C2907218; PART_NO (none) -> FRC0805F1000TS; PRICE_UNIT (none) -> 0.0029
- R6, R7: DISTRIBUTOR (none) -> LCSC; MANUFACTURER (none) -> FOJAN; ORDER_NO (none) -> C2907264; PART_NO (none) -> FRC0805F4701TS; PRICE_UNIT (none) -> 0,0026
- R9: DISTRIBUTOR (none) -> LCSC; MANUFACTURER (none) -> FOJAN; ORDER_NO (none) -> C2933415; PART_NO (none) -> FRC0805F3302TS; PRICE_UNIT (none) -> 0.0028
- SW1: DISTRIBUTOR (none) -> LCSC; MANUFACTURER (none) -> CAX; ORDER_NO (none) -> C53431127; PART_NO (none) -> TS-6645DD-6x6x5-100; PRICE_UNIT (none) -> 0.0361
- U1: DISTRIBUTOR (none) -> LCSC; MANUFACTURER (none) -> ST; ORDER_NO (none) -> C5456207; PART_NO (none) -> STM32C031C4T6; PRICE_UNIT (none) -> 1.5362
- U2, U3: DISTRIBUTOR (none) -> LCSC; MANUFACTURER (none) -> TI; ORDER_NO (none) -> C2841849; PART_NO (none) -> TMCS1100A4QDR; PRICE_UNIT (none) -> 3.2476
- U4: DISTRIBUTOR (none) -> LCSC; MANUFACTURER (none) -> TI; ORDER_NO (none) -> C130026; PART_NO (none) -> TCA9548APWR; PRICE_UNIT (none) -> 0.7641
- U5: DISTRIBUTOR (none) -> LCSC; ORDER_NO (none) -> C50278; PART_NO (none) -> MPU-6500; PRICE_UNIT (none) -> 4.9483
- U7: DISTRIBUTOR (none) -> LCSC; MANUFACTURER (none) -> ST; ORDER_NO (none) -> C672117; PART_NO (none) -> LD1117V33C; PRICE_UNIT (none) -> 0.59
- V1: DISTRIBUTOR MOUSER -> LCSC; MANUFACTURER Diotec -> onsemi; ORDER_NO 637-1n4148 -> C258182; PRICE_UNIT (none) -> 0.0272
Other:
- note removed: "Lap Sensor BOTTOM SIDE"
